File: hardware/kicad_proj/factory/perfect_console.kicad_sch (KiCad schematic)
At the start: 66 parts, among them J1 USB, J10 I2C, J11 ESP_UART, J12 CH_UART, J13 CH_Flash, J14 Micro_SD_Card, J16 DISP_MISO, J2 TP4056_WO_Protect, J3 Bat, J4 PWR_Btn, J5 BTNS, J6 PTT_Btn, J7 PWR_OUT, J8 40-41, J9 USB_Data, Q1 NMOS, Q2 NMOS, Q3 NMOS, Q4 NMOS, Q5 NMOS, Q6 NMOS, SW1 Reset, SW2 Boot, U1 ESP32-S3-WROOM1, U2 Display, U3 PCM5102, U4 CH32V006E8R6, U5 LoRa, U6 USBLC6-2SC6, U7 Mic, U8 DC-DC

Commit message: Покращення PCB
Parts:
- added C13: 10uF, Capacitor_SMD:C_1206_3216Metric_Pad1.33x1.80mm_HandSolder, symbol Device:C_Small
- C1, C10, C11, C12, C2, C3, C6, C7, C8, C9: footprint Capacitor_SMD:C_1206_3216Metric -> Capacitor_SMD:C_1206_3216Metric_Pad1.33x1.80mm_HandSolder
- C4: value 20uF -> 10uF; footprint Capacitor_SMD:C_1206_3216Metric -> Capacitor_SMD:C_1206_3216Metric_Pad1.33x1.80mm_HandSolder
- C5: value 0.1uF -> 100nF; footprint Capacitor_SMD:C_1206_3216Metric -> Capacitor_SMD:C_1206_3216Metric_Pad1.33x1.80mm_HandSolder
Connections:
- net +4V2: now also C13.1
- net at C4.2, C5.2, Q3.3 (D)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: now also C13.2
Changed lines of the file:
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@@
 	)
 	(junction
+		(at 330.2 354.33)
+		(diameter 0)
+		(color 0 0 0 0)
+	)
+	(junction
 		(at 243.84 228.6)
 		(diameter 0)
@@
 	(wire
 		(pts
+			(xy 326.39 354.33) (xy 330.2 354.33)
+		)
+		(stroke
+			(width 0)
+			(type default)
+		)
+	)
+	(wire
+		(pts
 			(xy 422.91 341.63) (xy 441.96 341.63)
 		)
@@
 	(wire
 		(pts
+			(xy 317.5 354.33) (xy 321.31 354.33)
+		)
+		(stroke
+			(width 0)
+			(type default)
+		)
+	)
+	(wire
+		(pts
 			(xy 640.08 379.73) (xy 646.43 379.73)
 		)
@@
 	(wire
 		(pts
+			(xy 330.2 354.33) (xy 330.2 360.68)
+		)
+		(stroke
+			(width 0)
+			(type default)
+		)
+	)
+	(wire
+		(pts
 			(xy 508 365.76) (xy 511.81 365.76)
 		)
@@
 	(wire
 		(pts
-			(xy 330.2 350.52) (xy 330.2 360.68)
+			(xy 330.2 350.52) (xy 330.2 354.33)
 		)
 		(stroke
@@
 			)
 		)
-		(property "Footprint" "Capacitor_SMD:C_1206_3216Metric"
+		(property "Footprint" "Capacitor_SMD:C_1206_3216Metric_Pad1.33x1.80mm_HandSolder"
 			(at 727.71 246.38 0)
 			(effects
@@
 			)
 		)
-		(property "Footprint" "Capacitor_SMD:C_1206_3216Metric"
+		(property "Footprint" "Capacitor_SMD:C_1206_3216Metric_Pad1.33x1.80mm_HandSolder"
 			(at 256.54 247.65 0)
 			(effects
@@
 		(dnp no)
 		(property "Reference" "C5"
-			(at 323.342 364.998 90)
+			(at 323.088 364.744 90)
 			(effects
 				(font
@@
 			)
 		)
-		(property "Value" "0.1uF"
-			(at 329.692 364.998 90)
+		(property "Value" "100nF"
+			(at 330.454 364.49 90)
 			(effects
 				(font
@@
 			)
 		)
-		(property "Footprint" "Capacitor_SMD:C_1206_3216Metric"
+		(property "Footprint" "Capacitor_SMD:C_1206_3216Metric_Pad1.33x1.80mm_HandSolder"
 			(at 323.85 367.03 0)
 			(effects
@@
 			)
 		)
-		(property "Value" "20uF"
+		(property "Value" "10uF"
 			(at 329.438 358.648 90)
 			(effects
@@
 			)
 		)
-		(property "Footprint" "Capacitor_SMD:C_1206_3216Metric"
+		(property "Footprint" "Capacitor_SMD:C_1206_3216Metric_Pad1.33x1.80mm_HandSolder"
 			(at 323.85 360.68 0)
 			(effects
@@
 			)
 		)
-		(property "Footprint" "Capacitor_SMD:C_1206_3216Metric"
+		(property "Footprint" "Capacitor_SMD:C_1206_3216Metric_Pad1.33x1.80mm_HandSolder"
 			(at 158.75 199.39 0)
 			(effects
@@
 			)
 		)
-		(property "Footprint" "Capacitor_SMD:C_1206_3216Metric"
+		(property "Footprint" "Capacitor_SMD:C_1206_3216Metric_Pad1.33x1.80mm_HandSolder"
 			(at 727.71 238.76 0)
 			(effects
@@
 	(symbol
 		(lib_id "power:+3V3")
+		(at 317.5 354.33 90)
+		(unit 1)
+		(exclude_from_sim no)
+		(in_bom yes)
+		(on_board yes)
+		(dnp no)
+		(property "Reference" "#PWR51"
+			(at 321.31 354.33 0)
+			(effects
+				(font
+					(size 1.27 1.27)
+				)
+				(hide yes)
+			)
+		)
+		(property "Value" "+4V2"
+			(at 312.674 354.33 90)
+			(effects
+				(font
+					(size 0.762 0.762)
+				)
+			)
+		)
+		(property "Footprint" ""
+			(at 317.5 354.33 0)
+			(effects
+				(font
+					(size 1.27 1.27)
+				)
+				(hide yes)
+			)
+		)
+		(property "Datasheet" ""
+			(at 317.5 354.33 0)
+			(effects
+				(font
+					(size 1.27 1.27)
+				)
+				(hide yes)
+			)
+		)
+		(property "Description" "Power symbol creates a global label with name \"+3V3\""
+			(at 317.5 354.33 0)
+			(effects
+				(font
+					(size 1.27 1.27)
+				)
+				(hide yes)
+			)
+		)
+		(pin "1"
+		)
+		(instances
+			(project "perfect_console"
+				(path "/17a56aab-f3dd-4de8-8a87-5e0772eddd26"
+					(reference "#PWR51")
+					(unit 1)
+				)
+			)
+		)
+	)
+	(symbol
+		(lib_id "Device:C_Small")
+		(at 323.85 354.33 90)
+		(unit 1)
+		(exclude_from_sim no)
+		(in_bom yes)
+		(on_board yes)
+		(dnp no)
+		(property "Reference" "C13"
+			(at 323.342 352.298 90)
+			(effects
+				(font
+					(size 1.27 1.27)
+				)
+				(justify left)
+			)
+		)
+		(property "Value" "10uF"
+			(at 329.438 352.298 90)
+			(effects
+				(font
+					(size 1.27 1.27)
+				)
+				(justify left)
+			)
+		)
+		(property "Footprint" "Capacitor_SMD:C_1206_3216Metric_Pad1.33x1.80mm_HandSolder"
+			(at 323.85 354.33 0)
+			(effects
+				(font
+					(size 1.27 1.27)
+				)
+				(hide yes)
+			)
+		)
+		(property "Datasheet" "~"
+			(at 323.85 354.33 0)
+			(effects
+				(font
+					(size 1.27 1.27)
+				)
+				(hide yes)
+			)
+		)
+		(property "Description" "Unpolarized capacitor, small symbol"
+			(at 323.85 354.33 0)
+			(effects
+				(font
+					(size 1.27 1.27)
+				)
+				(hide yes)
+			)
+		)
+		(pin "1"
+		)
+		(pin "2"
+		)
+		(instances
+			(project "perfect_console"
+				(path "/17a56aab-f3dd-4de8-8a87-5e0772eddd26"
+					(reference "C13")
+					(unit 1)
+				)
+			)
+		)
+	)
+	(symbol
+		(lib_id "power:+3V3")
 		(at 317.5 360.68 90)
 		(unit 1)
@@
 			)
 		)
-		(property "Footprint" "Capacitor_SMD:C_1206_3216Metric"
+		(property "Footprint" "Capacitor_SMD:C_1206_3216Metric_Pad1.33x1.80mm_HandSolder"
 			(at 400.05 339.09 0)
 			(effects
@@
 			)
 		)
-		(property "Footprint" "Capacitor_SMD:C_1206_3216Metric"
+		(property "Footprint" "Capacitor_SMD:C_1206_3216Metric_Pad1.33x1.80mm_HandSolder"
 			(at 515.62 223.52 0)
 			(effects
@@
 			)
 		)
-		(property "Footprint" "Capacitor_SMD:C_1206_3216Metric"
+		(property "Footprint" "Capacitor_SMD:C_1206_3216Metric_Pad1.33x1.80mm_HandSolder"
 			(at 558.8 215.9 0)
 			(effects
@@
 			)
 		)
-		(property "Footprint" "Capacitor_SMD:C_1206_3216Metric"
+		(property "Footprint" "Capacitor_SMD:C_1206_3216Metric_Pad1.33x1.80mm_HandSolder"
 			(at 652.78 350.52 0)
 			(effects
@@
 			)
 		)
-		(property "Footprint" "Capacitor_SMD:C_1206_3216Metric"
+		(property "Footprint" "Capacitor_SMD:C_1206_3216Metric_Pad1.33x1.80mm_HandSolder"
 			(at 436.88 207.01 0)
 			(effects
@@
 			)
 		)
-		(property "Footprint" "Capacitor_SMD:C_1206_3216Metric"
+		(property "Footprint" "Capacitor_SMD:C_1206_3216Metric_Pad1.33x1.80mm_HandSolder"
 			(at 158.75 194.31 0)
 			(effects

Commit message: Видалено ESD мікросхему та її конденсатор
Parts:
- removed C7: 100nF, Capacitor_SMD:C_1206_3216Metric_Pad1.33x1.80mm_HandSolder, symbol Device:C_Small
- removed U6: USBLC6-2SC6, Package_TO_SOT_SMD:SOT-23-6, symbol USBLC6-2SC6:USBLC6-2SC6
Other:
- moved on the sheet: C11, C12, C8, C9, Q5, Q6, R11, R12, R13, R14, R15, R16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

Commit message: Додано маркування мосфетів
Parts:
- Q1, Q2, Q3, Q4, Q5, Q6: value NMOS -> A09T
Changed lines of the file:
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@@
 			)
 		)
-		(property "Value" "NMOS"
+		(property "Value" "A09T"
 			(at 243.84 370.8399 0)
 			(effects
@@
 			)
 		)
-		(property "Value" "NMOS"
+		(property "Value" "A09T"
 			(at 448.3099 337.82 0)
 			(effects
@@
 			)
 		)
-		(property "Value" "NMOS"
+		(property "Value" "A09T"
 			(at 588.0101 209.55 0)
 			(effects
@@
 			)
 		)
-		(property "Value" "NMOS"
+		(property "Value" "A09T"
 			(at 158.75 377.1899 0)
 			(effects
@@
 			)
 		)
-		(property "Value" "NMOS"
+		(property "Value" "A09T"
 			(at 339.0899 363.22 0)
 			(effects
@@
 			)
 		)
-		(property "Value" "NMOS"
+		(property "Value" "A09T"
 			(at 562.6101 200.66 0)
 			(effects
